File: KiCad/$StereoAzimuthCorrector.sch (KiCad schematic (older format))
At the start: 36 parts

Commit message: Switch to low-power op-amp design
Parts:
- removed Q? (x2): NPN, symbol NPN
- removed R? (x2): 10k, symbol R
- added C? (x4): 470n, symbol C
- added R? (x5): 150k, symbol R
- added RV?: 100k, symbol POT
Connections:
- net GND: now also C?.2, C?.2, C?.2, C?.2, R?.2, RV?.3
- net VCC: now also C?.1, C?.1, R?.1, R?.1
- net VirtualGND: now also C?.1, R?.1, R?.2
- net at U?.12 (+): now also R?.1
- net at U?.13 (-): now also C?.1, R?.1
- new net: R?.2, RV?.1
- new net: R?.2, RV?.2
- new net +BATT: R?.2
Other:
- moved on the sheet: U?D
