File: KiCad/StereoAzimuthCorrector.sch (KiCad schematic (older format))
At the start: 51 parts, among them P1 12VDC_IN, P2 LR_OUT, P3 LR_OUT, P4 MONO_OUT, U1 TL064, U2 L78L09ACZ, U3 TL062

Commit message: Add part comments for ICs, diode, LED
Parts:
- D2: value DIODE -> 1N4148
- RV1: value B100K -> B100K_2
Other:
- note added: "D1: Osram LG R971-KN-1"
- note added: "D2: Fairchild LL4148\nU2: ST L78L09ACZ"
- note added: "ST TL062CDT"
- note added: "ST TL064CDT"
Changed lines of the file:
@@
 P 3700 2850
 F 0 "RV1" H 3860 3160 50  0000 C CNN
-F 1 "B100K" H 3990 2550 50  0000 C CNN
+F 1 "B100K_2" H 3990 2550 50  0000 C CNN
 F 2 "" H 3700 2850 60  0000 C CNN
 F 3 "" H 3700 2850 60  0000 C CNN
@@
 	5600 2950 6100 2950
 Wire Wire Line
-	7100 3050 7150 3050
-Wire Wire Line
-	7150 3050 7200 3050
+	7100 3050 7200 3050
 Wire Wire Line
 	7150 4000 7150 3050
 Connection ~ 6050 3150
 Wire Wire Line
-	6050 3150 6050 3350
-Wire Wire Line
-	6050 3350 6050 3450
-Wire Wire Line
-	6000 3150 6050 3150
-Wire Wire Line
-	6050 3150 6100 3150
+	6050 3150 6050 3450
+Wire Wire Line
+	6000 3150 6100 3150
 Connection ~ 4250 6300
 Wire Wire Line
@@
 Connection ~ 4600 6300
 Wire Wire Line
-	3200 6300 3250 6300
-Wire Wire Line
-	3250 6300 3550 6300
-Wire Wire Line
-	3550 6300 3900 6300
-Wire Wire Line
-	3900 6300 4250 6300
-Wire Wire Line
-	4250 6300 4600 6300
+	3200 6300 4600 6300
 Wire Wire Line
 	3900 6700 3900 6300
@@
 Connection ~ 4850 6900
 Wire Wire Line
-	4600 6250 4600 6300
-Wire Wire Line
-	4600 6300 4600 6350
+	4600 6250 4600 6350
 Connection ~ 4600 6900
 Wire Wire Line
 	4850 6900 4850 7000
 Wire Wire Line
-	4600 6900 4850 6900
-Wire Wire Line
-	4850 6900 5350 6900
-Wire Wire Line
-	4600 6850 4600 6900
-Wire Wire Line
-	4600 6900 4600 6950
+	4600 6900 5350 6900
+Wire Wire Line
+	4600 6850 4600 6950
 Connection ~ 4600 7500
 Wire Wire Line
 	4850 7500 4850 7400
 Wire Wire Line
-	1450 7500 1500 7500
-Wire Wire Line
-	1500 7500 1750 7500
-Wire Wire Line
-	1750 7500 2050 7500
-Wire Wire Line
-	2050 7500 2350 7500
-Wire Wire Line
-	2350 7500 2800 7500
-Wire Wire Line
-	2800 7500 3250 7500
-Wire Wire Line
-	3250 7500 3550 7500
-Wire Wire Line
-	3550 7500 3900 7500
-Wire Wire Line
-	3900 7500 4250 7500
-Wire Wire Line
-	4250 7500 4600 7500
-Wire Wire Line
-	4600 7500 4850 7500
-Wire Wire Line
-	4600 7450 4600 7500
-Wire Wire Line
-	4600 7500 4600 7550
+	1450 7500 4850 7500
+Wire Wire Line
+	4600 7450 4600 7550
 Connection ~ 6550 1200
 Connection ~ 6550 4450
@@
 	6000 4450 6100 4450
 Wire Wire Line
-	6500 4450 6550 4450
-Wire Wire Line
-	6550 4450 6850 4450
+	6500 4450 6850 4450
 Wire Wire Line
 	6550 4500 6550 4450
@@
 	6550 1200 6550 1250
 Wire Wire Line
-	6500 1200 6550 1200
-Wire Wire Line
-	6550 1200 6850 1200
+	6500 1200 6850 1200
 Wire Wire Line
 	6000 1200 6100 1200
@@
 	4350 4550 4400 4550
 Wire Wire Line
-	4350 4550 4350 5100
-Wire Wire Line
-	4350 5100 4350 5300
+	4350 4550 4350 5300
 Wire Wire Line
 	4650 5100 4350 5100
 Wire Wire Line
-	5400 4450 5450 4450
-Wire Wire Line
-	5450 4450 5500 4450
-Wire Wire Line
-	5450 3350 5450 4450
-Wire Wire Line
-	5450 4450 5450 5100
+	5400 4450 5500 4450
+Wire Wire Line
+	5450 3350 5450 5100
 Wire Wire Line
 	5450 5100 5150 5100
@@
 	4350 1300 4400 1300
 Wire Wire Line
-	4350 1300 4350 1850
-Wire Wire Line
-	4350 1850 4350 2050
+	4350 1300 4350 2050
 Wire Wire Line
 	4650 1850 4350 1850
 Wire Wire Line
-	5400 1200 5450 1200
-Wire Wire Line
-	5450 1200 5500 1200
+	5400 1200 5500 1200
 Wire Wire Line
 	5150 1850 5450 1850
@@
 	3550 2750 3250 2750
 Wire Wire Line
-	3250 1250 3250 2750
-Wire Wire Line
-	3250 2750 3250 2950
+	3250 1250 3250 2950
 Wire Wire Line
 	3250 2950 3550 2950
@@
 	2000 4900 2000 4850
 Wire Wire Line
-	2600 4450 2650 4450
-Wire Wire Line
-	2650 4450 3250 4450
+	2600 4450 3250 4450
 Wire Wire Line
 	2650 4450 2650 5200
@@
 	1400 4350 1400 4650
 Wire Wire Line
-	1350 4550 1550 4550
-Wire Wire Line
-	1550 4550 1600 4550
-Wire Wire Line
-	1350 4350 1400 4350
-Wire Wire Line
-	1400 4350 1600 4350
+	1350 4550 1600 4550
+Wire Wire Line
+	1350 4350 1600 4350
 Wire Wire Line
 	2000 2350 2000 2400
@@
 	2000 3250 2000 3200
 Wire Wire Line
-	2600 2800 2650 2800
-Wire Wire Line
-	2650 2800 3050 2800
+	2600 2800 3050 2800
 Wire Wire Line
 	2650 2800 2650 3550
@@
 	1400 2700 1400 3000
 Wire Wire Line
-	1350 2900 1550 2900
-Wire Wire Line
-	1550 2900 1600 2900
-Wire Wire Line
-	1350 2700 1400 2700
-Wire Wire Line
-	1400 2700 1600 2700
+	1350 2900 1600 2900
+Wire Wire Line
+	1350 2700 1600 2700
 Connection ~ 2650 1250
 Wire Wire Line
@@
 	2000 800  2000 850
 Wire Wire Line
-	2600 1250 2650 1250
-Wire Wire Line
-	2650 1250 3250 1250
+	2600 1250 3250 1250
 Wire Wire Line
 	2650 2000 2650 1250
@@
 	1400 1350 1600 1350
 Wire Wire Line
-	1400 1250 1400 1350
-Wire Wire Line
-	1400 1350 1400 1450
-Wire Wire Line
-	1400 1450 1400 1500
+	1400 1250 1400 1500
 Wire Wire Line
 	2000 1700 2000 1650
@@
 	5450 3150 5500 3150
 Wire Wire Line
-	5450 1200 5450 1850
-Wire Wire Line
-	5450 1850 5450 3150
+	5450 1200 5450 3150
 Wire Wire Line
 	5500 3350 5450 3350
@@
 Connection ~ 3550 6300
 Wire Wire Line
-	3250 5900 3250 6300
-Wire Wire Line
-	3250 6300 3250 6700
+	3250 5900 3250 6700
 Connection ~ 3250 6300
 Text Notes 3700 6300 0    60   ~ 0
@@
 Connection ~ 2350 7500
 Wire Wire Line
-	2350 5900 2350 6300
-Wire Wire Line
-	2350 6300 2350 6700
-Wire Wire Line
-	1450 6300 1500 6300
-Wire Wire Line
-	1500 6300 1750 6300
-Wire Wire Line
-	1750 6300 2050 6300
-Wire Wire Line
-	2050 6300 2350 6300
-Wire Wire Line
-	2350 6300 2400 6300
+	2350 5900 2350 6700
+Wire Wire Line
+	1450 6300 2400 6300
 Wire Wire Line
 	2050 6700 2050 6300
@@
 P 2800 5900
 F 0 "D2" H 2800 6000 50  0000 C CNN
-F 1 "DIODE" H 2800 5800 50  0000 C CNN
+F 1 "1N4148" H 2800 5800 50  0000 C CNN
 F 2 "" H 2800 5900 60  0000 C CNN
 F 3 "" H 2800 5900 60  0000 C CNN
@@
 	1400 6850 1500 6850
 Wire Wire Line
-	1500 6850 1500 6950
-Wire Wire Line
-	1500 6950 1500 7500
+	1500 6850 1500 7500
 Connection ~ 1750 7500
 Wire Wire Line
@@
 $EndComp
 Wire Wire Line
-	9700 2000 9700 2050
-Wire Wire Line
-	9700 2050 9700 2100
+	9700 2000 9700 2100
 $Comp
 L RCJ-2223 P2
@@
 $EndComp
 Wire Wire Line
-	8800 2050 9700 2050
-Wire Wire Line
-	9700 2050 10200 2050
+	8800 2050 10200 2050
 Wire Wire Line
 	8800 2050 8800 2000
@@
 	10000 1450 10250 1450
 Wire Wire Line
-	8200 3050 8250 3050
-Wire Wire Line
-	8250 3050 8550 3050
+	8200 3050 8550 3050
 Wire Wire Line
 	10250 1550 10200 1550
@@
 Connection ~ 1500 6300
 Connection ~ 1500 7500
+Text Notes 2050 1000 0    60   ~ 0
+ST TL064CDT
+Text Notes 4850 950  0    60   ~ 0
+ST TL062CDT
+Text Notes 2350 5750 0    60   ~ 0
+D2: Fairchild LL4148\nU2: ST L78L09ACZ
+Text Notes 1700 7650 0    60   ~ 0
+D1: Osram LG R971-KN-1
 $EndSCHEMATC

Commit message: Finalize component choice, add datasheets
Parts:
- removed C12, C13, C14, C3, C6: 10u, symbol C
- removed P2, P3: LR_OUT, symbol RCJ-2223
- added C12, C13, C14, C3, C6: 10u, Capacitors_Elko_ThroughHole:Elko_vert_11x5mm_RM2, symbol CP1
- added C15, C16: 470n, Capacitors_SMD:C_1206_HandSoldering, symbol C
- added P2, P3: SAC_P_3.5MM, symbol SAC_P_3.5MM
- added P5, P6, P7, P8: HOLE, Mounting_Holes:MountingHole_2-5mm, symbol CONN_01X01
- C1, C10, C11, C2, C4, C5, C7, C8, C9: footprint (none) -> Capacitors_SMD:C_1206_HandSoldering
- D1: footprint (none) -> LEDs:LED-5MM
- D2: footprint (none) -> Discret:DO-35
- P1: footprint (none) -> Oddities:Dummy_Empty
- P4: footprint (none) -> Pin_Headers:Pin_Header_Straight_1x02
- R1, R11, R12, R13, R14, R15, R16, R17, R18, R19, R2, R20, R21, R22, R23, R24, R25, R26, R27, R3, R4, R5, R6, R7, R8, R9: footprint (none) -> Resistors_SMD:R_1206_HandSoldering
- R10: value 2.2k -> 1.2k; footprint (none) -> Resistors_SMD:R_1206_HandSoldering
- RV1: value B100K_2 -> B50K_2
- U1: footprint (none) -> Housings_SOIC:SOIC-14_3.9x8.7mm_Pitch1.27mm
- U2: footprint TO-92 -> Housings_TO-92:TO-92_Molded_Narrow
- U3: footprint (none) -> Housings_SOIC:SOIJ-8_5.3x5.3mm_Pitch1.27mm
Connections:
- net GND: now also C3.2, C6.2, P2.5, P3.5
- net L'+R': now also C14.2
- net L_in: now also C16.2
- net R_in: now also C15.2
- net VCC: now also C6.1
- net ~L'~_out: now also C12.2, P3.4
- net ~R'~_out: now also C13.2, P3.1
- net at R19.1: now also C12.1
- net at R22.1: now also C13.1
- net at R26.1: now also C14.1
- net at C4.1, D2.2 (K), P1.1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: now also C3.1
- new net: C15.1, P2.1
- new net: C16.1, P2.4
- no-connect marks 0 -> 4
Other:
- note added: "2x Switchcraft 35RASMT2BHNTRX"
- note added: "No place"
- note added: "U2: ST L78L09ACZ"
- note removed: "CUI RCJ-2223"
- note removed: "D1: Osram LG R971-KN-1"
- note removed: "D2: Fairchild LL4148\nU2: ST L78L09ACZ"
- moved on the sheet: P4

Commit message: Rough in component placement
Power jack footprint is still TODO
Parts:
- D1: footprint LEDs:LED-5MM -> SAC_footprints:SAC_LED-5MM
- D2: footprint Discret:DO-35 -> SAC_footprints:SAC_DO-35
- P1: footprint Oddities:Dummy_Empty -> Connect:BARREL_JACK
- P2, P3: footprint (none) -> SAC_footprints:SAC_P_3.5MM
- RV1: footprint (none) -> SAC_footprints:SAC_RV1
Changed lines of the file:
@@
 $EndComp
 $Comp
-L GND #PWR4
+L GND #PWR01
 U 1 1 559C0E9D
 P 2000 1700
-F 0 "#PWR4" H 2000 1450 60  0001 C CNN
+F 0 "#PWR01" H 2000 1450 60  0001 C CNN
 F 1 "GND" H 2000 1550 60  0000 C CNN
 F 2 "" H 2000 1700 60  0000 C CNN
@@
 $EndComp
 $Comp
-L VCC #PWR3
+L VCC #PWR02
 U 1 1 559C1056
 P 2000 800
-F 0 "#PWR3" H 2000 650 60  0001 C CNN
+F 0 "#PWR02" H 2000 650 60  0001 C CNN
 F 1 "VCC" H 2000 950 60  0000 C CNN
 F 2 "" H 2000 800 60  0000 C CNN
@@
 $EndComp
 $Comp
-L GND #PWR1
+L GND #PWR03
 U 1 1 559C1835
 P 1400 4000
-F 0 "#PWR1" H 1400 3750 60  0001 C CNN
+F 0 "#PWR03" H 1400 3750 60  0001 C CNN
 F 1 "GND" H 1400 3850 60  0000 C CNN
 F 2 "" H 1400 4000 60  0000 C CNN
@@
 $EndComp
 $Comp
-L GND #PWR6
+L GND #PWR04
 U 1 1 559C1A09
 P 2000 3250
-F 0 "#PWR6" H 2000 3000 60  0001 C CNN
+F 0 "#PWR04" H 2000 3000 60  0001 C CNN
 F 1 "GND" H 2000 3100 60  0000 C CNN
 F 2 "" H 2000 3250 60  0000 C CNN
@@
 $EndComp
 $Comp
-L VCC #PWR5
+L VCC #PWR05
 U 1 1 559C1CC3
 P 2000 2350
-F 0 "#PWR5" H 2000 2200 60  0001 C CNN
+F 0 "#PWR05" H 2000 2200 60  0001 C CNN
 F 1 "VCC" H 2000 2500 60  0000 C CNN
 F 2 "" H 2000 2350 60  0000 C CNN
@@
 $EndComp
 $Comp
-L GND #PWR2
+L GND #PWR06
 U 1 1 559C221F
 P 1400 5650
-F 0 "#PWR2" H 1400 5400 60  0001 C CNN
+F 0 "#PWR06" H 1400 5400 60  0001 C CNN
 F 1 "GND" H 1400 5500 60  0000 C CNN
 F 2 "" H 1400 5650 60  0000 C CNN
@@
 $EndComp
 $Comp
-L GND #PWR8
+L GND #PWR07
 U 1 1 559C222A
 P 2000 4900
-F 0 "#PWR8" H 2000 4650 60  0001 C CNN
+F 0 "#PWR07" H 2000 4650 60  0001 C CNN
 F 1 "GND" H 2000 4750 60  0000 C CNN
 F 2 "" H 2000 4900 60  0000 C CNN
@@
 $EndComp
 $Comp
-L VCC #PWR7
+L VCC #PWR08
 U 1 1 559C2233
 P 2000 4000
-F 0 "#PWR7" H 2000 3850 60  0001 C CNN
+F 0 "#PWR08" H 2000 3850 60  0001 C CNN
 F 1 "VCC" H 2000 4150 60  0000 C CNN
 F 2 "" H 2000 4000 60  0000 C CNN
@@
 F 0 "RV1" H 3860 3160 50  0000 C CNN
 F 1 "B50K_2" H 3990 2550 50  0000 C CNN
-F 2 "" H 3700 2850 60  0001 C CNN
+F 2 "SAC_footprints:SAC_RV1" H 3700 2850 60  0001 C CNN
 F 3 "" H 3700 2850 60  0000 C CNN
 	1    3700 2850
@@
 $EndComp
 $Comp
-L GND #PWR15
+L GND #PWR09
 U 1 1 559C3CF6
 P 5200 2550
-F 0 "#PWR15" H 5200 2300 60  0001 C CNN
+F 0 "#PWR09" H 5200 2300 60  0001 C CNN
 F 1 "GND" H 5200 2400 60  0000 C CNN
 F 2 "" H 5200 2550 60  0000 C CNN
@@
 $EndComp
 $Comp
-L VCC #PWR11
+L VCC #PWR010
 U 1 1 559C43F2
 P 4800 750
-F 0 "#PWR11" H 4800 600 60  0001 C CNN
+F 0 "#PWR010" H 4800 600 60  0001 C CNN
 F 1 "VCC" H 4800 900 60  0000 C CNN
 F 2 "" H 4800 750 60  0000 C CNN
@@
 $EndComp
 $Comp
-L GND #PWR12
+L GND #PWR011
 U 1 1 559C4721
 P 4800 1650
-F 0 "#PWR12" H 4800 1400 60  0001 C CNN
+F 0 "#PWR011" H 4800 1400 60  0001 C CNN
 F 1 "GND" H 4950 1600 60  0000 C CNN
 F 2 "" H 4800 1650 60  0000 C CNN
@@
 $EndComp
 $Comp
-L GND #PWR16
+L GND #PWR012
 U 1 1 559C4F96
 P 5200 5800
-F 0 "#PWR16" H 5200 5550 60  0001 C CNN
+F 0 "#PWR012" H 5200 5550 60  0001 C CNN
 F 1 "GND" H 5200 5650 60  0000 C CNN
 F 2 "" H 5200 5800 60  0000 C CNN
@@
 $EndComp
 $Comp
-L VCC #PWR13
+L VCC #PWR013
 U 1 1 559C4FA9
 P 4800 4000
-F 0 "#PWR13" H 4800 3850 60  0001 C CNN
+F 0 "#PWR013" H 4800 3850 60  0001 C CNN
 F 1 "VCC" H 4800 4150 60  0000 C CNN
 F 2 "" H 4800 4000 60  0000 C CNN
@@
 $EndComp
 $Comp
-L GND #PWR14
+L GND #PWR014
 U 1 1 559C4FB0
 P 4800 4900
-F 0 "#PWR14" H 4800 4650 60  0001 C CNN
+F 0 "#PWR014" H 4800 4650 60  0001 C CNN
 F 1 "GND" H 4950 4850 60  0000 C CNN
 F 2 "" H 4800 4900 60  0000 C CNN
@@
 $EndComp
 $Comp
-L GND #PWR19
+L GND #PWR015
 U 1 1 559C6192
 P 6550 1800
-F 0 "#PWR19" H 6550 1550 60  0001 C CNN
+F 0 "#PWR015" H 6550 1550 60  0001 C CNN
 F 1 "GND" H 6550 1650 60  0000 C CNN
 F 2 "" H 6550 1800 60  0000 C CNN
@@
 $EndComp
 $Comp
-L GND #PWR20
+L GND #PWR016
 U 1 1 559C667D
 P 6550 5050
-F 0 "#PWR20" H 6550 4800 60  0001 C CNN
+F 0 "#PWR016" H 6550 4800 60  0001 C CNN
 F 1 "GND" H 6550 4900 60  0000 C CNN
 F 2 "" H 6550 5050 60  0000 C CNN
@@
 $EndComp
 $Comp
-L GND #PWR10
+L GND #PWR017
 U 1 1 559CE992
 P 4600 7550
-F 0 "#PWR10" H 4600 7300 60  0001 C CNN
+F 0 "#PWR017" H 4600 7300 60  0001 C CNN
 F 1 "GND" H 4600 7400 60  0000 C CNN
 F 2 "" H 4600 7550 60  0000 C CNN
@@
 $EndComp
 $Comp
-L VCC #PWR9
+L VCC #PWR018
 U 1 1 559CECCA
 P 4600 6250
-F 0 "#PWR9" H 4600 6100 60  0001 C CNN
+F 0 "#PWR018" H 4600 6100 60  0001 C CNN
 F 1 "VCC" H 4600 6400 60  0000 C CNN
 F 2 "" H 4600 6250 60  0000 C CNN
@@
 F 0 "D1" H 1700 7050 50  0000 C CNN
 F 1 "PWR_ON" H 1750 7250 50  0000 C CNN
-F 2 "LEDs:LED-5MM" H 1750 7150 60  0001 C CNN
+F 2 "SAC_footprints:SAC_LED-5MM" H 1750 7150 60  0001 C CNN
 F 3 "" H 1750 7150 60  0000 C CNN
 	1    1750 7150
@@
 L'+R'
 $Comp
-L GND #PWR18
+L GND #PWR019
 U 1 1 559DBA4C
 P 6500 3500
-F 0 "#PWR18" H 6500 3250 60  0001 C CNN
+F 0 "#PWR019" H 6500 3250 60  0001 C CNN
 F 1 "GND" H 6500 3350 60  0000 C CNN
 F 2 "" H 6500 3500 60  0000 C CNN
@@
 $EndComp
 $Comp
-L VCC #PWR17
+L VCC #PWR020
 U 1 1 559DBF3A
 P 6500 2600
-F 0 "#PWR17" H 6500 2450 60  0001 C CNN
+F 0 "#PWR020" H 6500 2450 60  0001 C CNN
 F 1 "VCC" H 6500 2750 60  0000 C CNN
 F 2 "" H 6500 2600 60  0000 C CNN
@@
 $EndComp
 $Comp
-L GND #PWR21
+L GND #PWR021
 U 1 1 559DDFF0
 P 8250 3700
-F 0 "#PWR21" H 8250 3450 60  0001 C CNN
+F 0 "#PWR021" H 8250 3450 60  0001 C CNN
 F 1 "GND" H 8250 3550 60  0000 C CNN
 F 2 "" H 8250 3700 60  0000 C CNN
@@
 F 0 "D2" H 2800 6000 50  0000 C CNN
 F 1 "1N4148" H 2800 5800 50  0000 C CNN
-F 2 "Discret:DO-35" H 2800 5900 60  0001 C CNN
+F 2 "SAC_footprints:SAC_DO-35" H 2800 5900 60  0001 C CNN
 F 3 "" H 2800 5900 60  0000 C CNN
 	1    2800 5900
@@
 F 0 "P1" H 1100 7100 60  0000 C CNN
 F 1 "12VDC_IN" H 1100 6650 60  0000 C CNN
-F 2 "Oddities:Dummy_Empty" H 1100 6850 60  0001 C CNN
+F 2 "Connect:BARREL_JACK" H 1100 6850 60  0001 C CNN
 F 3 "" H 1100 6850 60  0000 C CNN
 	1    1100 6850
@@
 	9150 5200 9450 5200
 $Comp
-L GND #PWR22
+L GND #PWR022
 U 1 1 559F667D
 P 9400 5950
-F 0 "#PWR22" H 9400 5700 60  0001 C CNN
+F 0 "#PWR022" H 9400 5700 60  0001 C CNN
 F 1 "GND" H 9400 5800 60  0000 C CNN
 F 2 "" H 9400 5950 60  0000 C CNN
@@
 CUI PJ-202A
 $Comp
-L PWR_FLAG #FLG2
+L PWR_FLAG #FLG023
 U 1 1 55A01C76
 P 1450 7500
-F 0 "#FLG2" H 1450 7595 30  0001 C CNN
+F 0 "#FLG023" H 1450 7595 30  0001 C CNN
 F 1 "PWR_FLAG" H 1450 7680 30  0000 C CNN
 F 2 "" H 1450 7500 60  0000 C CNN
@@
 $EndComp
 $Comp
-L PWR_FLAG #FLG1
+L PWR_FLAG #FLG024
 U 1 1 55A01CBF
 P 1450 6300
-F 0 "#FLG1" H 1450 6395 30  0001 C CNN
+F 0 "#FLG024" H 1450 6395 30  0001 C CNN
 F 1 "PWR_FLAG" H 1450 6480 30  0000 C CNN
 F 2 "" H 1450 6300 60  0000 C CNN
@@
 F 0 "P2" H 8100 5150 50  0000 C CNN
 F 1 "SAC_P_3.5MM" H 8250 5600 50  0000 C CNN
-F 2 "" H 8400 5350 60  0000 C CNN
+F 2 "SAC_footprints:SAC_P_3.5MM" H 8400 5350 60  0001 C CNN
 F 3 "" H 8400 5350 60  0000 C CNN
 	1    8400 5350
@@
 F 0 "P3" H 9450 5150 50  0000 C CNN
 F 1 "SAC_P_3.5MM" H 9600 5600 50  0000 C CNN
-F 2 "" H 9750 5350 60  0000 C CNN
+F 2 "SAC_footprints:SAC_P_3.5MM" H 9750 5350 60  0001 C CNN
 F 3 "" H 9750 5350 60  0000 C CNN
 	1    9750 5350
